File: eagle/Solar_Autoguider/main.brd (EAGLE design)
At the start: 51.7 x 73.7 mm, 13 parts, among them IC1 7805T, X1 PG203J, X2 YH-55-10

Commit message: Better silk-screen on board.
Changed lines of the file:
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@@
 <text x="7.62" y="50.8" size="1.778" layer="21">V+</text>
 <text x="15.24" y="46.99" size="1.778" layer="21">G</text>
-<text x="36.83" y="72.39" size="1.778" layer="21" rot="R270">LX50 Solar Autoguider
+<text x="22.86" y="64.77" size="1.778" layer="21" rot="R270">LX50 Solar Autoguider
 Rev. C
 Bryan Lunt, 2014/2015</text>
@@
 <element name="R4" library="resistor" package="0207/7" value="100" x="41.91" y="27.94"/>
 <element name="R_PU" library="resistor" package="0207/7" value="10000" x="12.7" y="41.91" rot="R270"/>
-<element name="U$1" library="Arduini_Nano" package="NANO_PACK" value="ARDUINO_NANO_DEV" x="26.67" y="49.53" rot="R180"/>
+<element name="U$1" library="Arduini_Nano" package="NANO_PACK" value="ARDUINO_NANO_DEV" x="26.67" y="49.53" smashed="yes" rot="R180"/>
 <element name="X1" library="con-hirschmann" package="PG203J" value="PG203J" x="7.62" y="7.62" rot="R90">
 <attribute name="OC_NEWARK" value="unknown" x="7.62" y="7.62" size="1.778" layer="27" rot="R90" display="off"/>
