File: eagle/Solar_Autoguider/main.sch (EAGLE design)
At the start: 13 parts, among them IC1 7805T, X1 PG203J, X2 YH-55-10

Commit message: Better silk-screen on board.
Parts:
- C1, JP1, JP2, R1, R2, R3, R4, R_PU, U$1: OC_NEWARK (none) -> unknown
- IC1: MPN (none) -> LM7805CT; OC_NEWARK (none) -> 34C1092
- X2: value YH-55-10 -> XRJK-S-01-6-6-0-2G2-NO; device con-wenzhou-yihua:YH-55-10 -> con-xmultiple:XRJK-S-01-6-6-0-2G2-NO; OC_NEWARK (none) -> unknown
